File: hardware/alarm-panel/Alarm Panel.kicad_pcb (KiCad board)
At the start: 2 copper layers, 110 x 80 mm, 34 parts, among them J1 DC_BARREL_JACK, J10 W5500, J11 AUX_12V_GND, J12 AUX_12V_GND, J13 SIREN_OUT, J2 Z1_GND_Z2, J3 Z3_GND_Z4, J4 Z5_GND_Z6, J5 Z7_GND_Z8, J6 Z9_GND_Z10, J7 SPARE_NC_GND_NC, J8 PWR_MODULE, J9 ESP32_OLED, Q1 IRFZ44N, U1 TC4420CPA

Commit message: Update PCB layout and organize project structure
Parts:
- moved C5 3.20 mm to (40.5, 56.0)
- moved C3 2.50 mm to (51.0, 60.5)
Routing:
- net 12V: track 251.3 -> 255.8 mm
- net GND: track 565.2 -> 567.9 mm
- net 3V3: track 126.8 -> 129.3 mm
Other:
- board text added: "Alarm Panel (OLED) by Gary Taylor v1.0.0"

Commit message: On branch Gerber-Files-Created Changes to be committed: 	modified:   docs/pcb/pcb-completion-checklist.md 	modified:   hardware/alarm-panel/Alarm Panel.kicad_pcb 	new file:   hardware/alarm-panel/gerbers/Alarm Panel-B_Cu.gbl 	new file:   hardware/alarm-panel/gerbers/Alarm Panel-B_Mask.gbs 	new file:   hardware/alarm-panel/gerbers/Alarm Panel-B_Silkscreen.gbo 	new file:   hardware/alarm-panel/gerbers/Alarm Panel-Edge_Cuts.gm1 	new file:   hardware/alarm-panel/gerbers/Alarm Panel-F_Cu.gtl 	new file:   hardware/alarm-panel/gerbers/Alarm Panel-F_Mask.gts 	new file:   hardware/alarm-panel/gerbers/Alarm Panel-F_Silkscreen.gto 	new file:   hardware/alarm-panel/gerbers/Alarm Panel-NPTH.drl 	new file:   hardware/alarm-panel/gerbers/Alarm Panel-PTH.drl 	new file:   hardware/alarm-panel/gerbers/Alarm Panel-job.gbrjob 	new file:   hardware/alarm-panel/gerbers/Alarm-Panel.zip
Routing:
- added copper zone on B.Cu, net GND
Changed lines of the file:
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@@
 		(filling no)
 		(pcbplotparams
-			(layerselection 0x00000000_00000000_55555555_5755f5ff)
+			(layerselection 0x00000000_00000000_55555555_575555ff)
 			(plot_on_all_layers_selection 0x00000000_00000000_00000000_00000000)
 			(disableapertmacros no)
-			(usegerberextensions no)
+			(usegerberextensions yes)
 			(usegerberattributes yes)
 			(usegerberadvancedattributes yes)
@@
 			(sketchdnponfab yes)
 			(crossoutdnponfab yes)
-			(subtractmaskfromsilk no)
+			(subtractmaskfromsilk yes)
 			(outputformat 1)
 			(mirror no)
-			(drillshape 1)
+			(drillshape 0)
 			(scaleselection 1)
-			(outputdirectory "")
+			(outputdirectory "gerbers/")
 		)
 	)
@@
 		(tags "THT terminal block 2.54mm 1x03")
 		(property "Reference" "J4"
-			(at 2.535 1.7 0)
+			(at 5.035 -6.8 0)
 			(layer "F.SilkS")
 			(effects
@@
 		(tags "THT terminal block 2.54mm 1x03")
 		(property "Reference" "J5"
-			(at 2.285 1.7 0)
+			(at 5.285 -6.8 0)
 			(layer "F.SilkS")
 			(effects
@@
 		(tags "THT terminal block 2.54mm 1x02")
 		(property "Reference" "J11"
-			(at 1.24 1.7 0)
+			(at -3.76 -0.8 0)
 			(layer "F.SilkS")
 			(effects
@@
 		(tags "THT terminal block 2.54mm 1x03")
 		(property "Reference" "J7"
-			(at 2.54 1.7 0)
+			(at 4.785 -6.8 0)
 			(layer "F.SilkS")
 			(effects
@@
 		(tags "THT terminal block 2.54mm 1x03")
 		(property "Reference" "J3"
-			(at 2.285 1.7 0)
+			(at 5.285 -6.8 0)
 			(layer "F.SilkS")
 			(effects
@@
 		(tags "THT terminal block 2.54mm 1x03")
 		(property "Reference" "J6"
-			(at 2.535 1.7 0)
+			(at 5.035 -6.8 0)
 			(layer "F.SilkS")
 			(effects
@@
 		(tags "THT terminal block 2.54mm 1x03")
 		(property "Reference" "J2"
-			(at 2.535 1.7 0)
+			(at 5.035 -6.8 0)
 			(layer "F.SilkS")
 			(effects
@@
 		(net "FUSED_12V")
 	)
+	(zone
+		(net "GND")
+		(layer "B.Cu")
+		(hatch edge 0.5)
+		(connect_pads
+			(clearance 0.5)
+		)
+		(min_thickness 0.25)
+		(fill yes
+			(thermal_gap 0.5)
+			(thermal_bridge_width 0.5)
+			(island_removal_mode 0)
+		)
+		(polygon
+			(pts
+				(xy 0 0) (xy 110 0) (xy 110 80) (xy 0 80)
+			)
+		)
+	)
 	(group ""
