File: hardware/alarm-panel/Alarm Panel.kicad_pcb (KiCad board)
At the start: 2 copper layers, 110 x 80 mm, 34 parts, among them J1 DC_BARREL_JACK, J10 W5500, J11 AUX_12V_GND, J12 AUX_12V_GND, J13 SIREN_OUT, J2 Z1_GND_Z2, J3 Z3_GND_Z4, J4 Z5_GND_Z6, J5 Z7_GND_Z8, J6 Z9_GND_Z10, J7 SPARE_NC_GND_NC, J8 PWR_MODULE, J9 ESP32_OLED, Q1 IRFZ44N, U1 TC4420CPA

Commit message: bump silkscreen version number on PCB.  Rename gerber zip file to include version and JLCPCB reference.
Other:
- board text added: "Alarm Panel (OLED) by Gary Taylor v1.1.0"
- board text removed: "Alarm Panel (OLED) by Gary Taylor v1.0.0"
Changed lines of the file:
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@@
 		)
 	)
-	(gr_text "Alarm Panel (OLED)\nby Gary Taylor\nv1.0.0"
+	(gr_text "Alarm Panel (OLED)\nby Gary Taylor\nv1.1.0"
 		(at 32.5 35 0)
 		(layer "F.SilkS")
